Commit message: trooooop d'erreur mais on garde un peu d'espoir, un tout petit peu

File: install/moveit_config/share/moveit_config/config/robot.ros2_control.xacro (robot description, xacro)
@@ -2,5 +2,5 @@
 <robot xmlns:xacro="http://www.ros.org/wiki/xacro">
     <xacro:macro name="robot_ros2_control" params="name initial_positions_file">
-        <xacro:property name="initial_positions" value="${xacro.load_yaml(initial_positions_file)['initial_positions']}"/>
+        <xacro:property name="initial_positions" value="${load_yaml(initial_positions_file)['initial_positions']}"/>
         <ros2_control name="${name}" type="system">
             <hardware>
@@ -8,4 +8,11 @@
                 <plugin>mock_components/GenericSystem</plugin>
             </hardware>
+            <joint name="Z_Translation">
+                <command_interface name="position"/>
+                <state_interface name="position">
+                  <param name="initial_value">${initial_positions['Z_Translation']}</param>
+                </state_interface>
+                <state_interface name="velocity"/>
+            </joint>
             <joint name="X_Translation">
                 <command_interface name="position"/>

File: install/urdf_tutorial/share/urdf_tutorial/urdf/robot.urdf (robot description, URDF)
Before this commit: robot robot, 5 links, 4 joints
Links:
- added link Trans_Z_Axes; collision box size=0.25 0.20 1; visual box size=0.25 0.20 1
- link Rotation_Part: geometry collision box size=0.035 0.035 0.035; visual box size=0.035 0.035 0.035
Joints:
- added joint Z_Translation: type prismatic, parent base_link, child Trans_Z_Axes, origin xyz=0 0 0, axis 0 0 1, limit lower=0 upper=0.550 effort=1000.0 velocity=0.5
- joint Rotation: origin xyz=0.045 0 0 -> xyz=0.04 0 0
- joint X_Translation: parent base_link -> Trans_Z_Axes

Commit message: abandon de MoveIt

File: install/moveit_config/share/moveit_config/config/robot.ros2_control.xacro (robot description, xacro)
@@ -2,5 +2,5 @@
 <robot xmlns:xacro="http://www.ros.org/wiki/xacro">
     <xacro:macro name="robot_ros2_control" params="name initial_positions_file">
-        <xacro:property name="initial_positions" value="${load_yaml(initial_positions_file)['initial_positions']}"/>
+        <xacro:property name="initial_positions" value="${xacro.load_yaml(initial_positions_file)['initial_positions']}"/>
         <ros2_control name="${name}" type="system">
             <hardware>

File: install/urdf_tutorial/share/urdf_tutorial/urdf/robot.urdf (robot description, URDF)
Before this commit: robot robot, 6 links, 5 joints
Joints:
- joint Rotation: axis (none) -> 0 1 0
